File: hardware/PCB/Scene_Display.kicad_sch (KiCad schematic)
At the start: 12 parts, among them U17 MAX7219, U18 SA15-11SRWA, U19 SA15-11SRWA, U20 SA15-11SRWA, U21 SA15-11SRWA, U22 SA15-11SRWA, U23 SA15-11SRWA, U24 SA15-11SRWA, U25 SA15-11SRWA

Commit message: change page structure
Parts:
- removed C19: 100nF/50V, Capacitor_SMD:C_1206_3216Metric_Pad1.33x1.80mm_HandSolder, symbol Device:C
- removed C20: 470uF/10V, Capacitor_Tantalum_SMD:CP_EIA-7343-31_Kemet-D_Pad2.25x2.55mm_HandSolder, symbol Device:C_Polarized
- removed RV4: 20K, Potentiometer_SMD:Potentiometer_Vishay_TS53YL_Vertical, symbol Device:R_Potentiometer_Trim
- removed U17: MAX7219, Package_SO:SOIC-24W_7.5x15.4mm_P1.27mm, symbol Driver_LED:MAX7219
- removed U18, U19, U20, U21, U22, U23, U24, U25: SA15-11SRWA, 7-segment-led:FYS-12011A, symbol Display_Character:SA15-11SRWA
Connections:
- no-connect marks 1 -> 0
Other:
- note removed: "Front LED Display"
