File: hardware/PCB/DigiSlatePlus.kicad_pcb (KiCad board)
At the start: 2 copper layers, 270 x 120 mm, 34 parts, among them J1 Barrel_Jack_MountingPin, J2 AudioJack3_SwitchTR, J3 PinHeader 2x3, Q1 2N2222, U1 ATmega328-A, U1 ESP32-S3-WROOM-1, U10 SA15-11SRWA, U2 MAX7219, U3 SA15-11SRWA, U4 SA15-11SRWA, U5 SA15-11SRWA, U6 SA15-11SRWA, U7 SA15-11SRWA, U8 SA15-11SRWA, U9 SA15-11SRWA, Y1 16 MHz

Commit message: TP4056 library added
Parts:
- removed J1: Barrel_Jack_MountingPin, Connector_BarrelJack:BarrelJack_GCT_DCJ200-10-A_Horizontal
- removed J2: AudioJack3_SwitchTR, Connector_Audio:Jack_3.5mm_CUI_SJ1-3525N_Horizontal
- removed J3: PinHeader 2x3, Connector_PinHeader_2.54mm:PinHeader_2x03_P2.54mm_Vertical
- removed the R1 at (107.5, 91.0)
- removed the R1 at (99.0, 92.5)
- removed the U1 at (87.8, 154.8)
- removed Y1: 16 MHz, Crystal:Resonator_SMD_Murata_CSTxExxV-3Pin_3.0x1.1mm_HandSoldering
- added C10: 10nF/50V, Capacitor_SMD:C_1206_3216Metric_Pad1.33x1.80mm_HandSolder, B.Cu at (127.5, 59.4)
- added C11: 100uF/10V, Capacitor_Tantalum_SMD:CP_EIA-7343-31_Kemet-D_Pad2.25x2.55mm_HandSolder, B.Cu at (121.8, 59.7)
- added C12: 10nF/50V, Capacitor_SMD:C_1206_3216Metric_Pad1.33x1.80mm_HandSolder, B.Cu at (27.0, 53.1)
- added C13: 220uF/25V, Capacitor_Tantalum_SMD:CP_EIA-7343-31_Kemet-D_Pad2.25x2.55mm_HandSolder, B.Cu at (20.8, 54.0)
- added C14: 100nF/50V, Capacitor_SMD:C_1206_3216Metric_Pad1.33x1.80mm_HandSolder, B.Cu at (101.2, 60.1)
- added C15: 220uF/10V, Capacitor_Tantalum_SMD:CP_EIA-7343-31_Kemet-D_Pad2.25x2.55mm_HandSolder, B.Cu at (106.0, 59.7)
- added C5: 10nF/50V, Capacitor_SMD:C_1206_3216Metric_Pad1.33x1.80mm_HandSolder, B.Cu at (35.8, 64.8)
- added C6: 100uF/10V, Capacitor_Tantalum_SMD:CP_EIA-7343-31_Kemet-D_Pad2.25x2.55mm_HandSolder, B.Cu at (123.5, 46.0)
- added C7: 220uF/25V, Capacitor_Tantalum_SMD:CP_EIA-7343-31_Kemet-D_Pad2.25x2.55mm_HandSolder, B.Cu at (35.5, 60.0)
- added C8: 100nF/50V, Capacitor_SMD:C_1206_3216Metric_Pad1.33x1.80mm_HandSolder, B.Cu at (101.5, 46.0)
- added C9: 220uF/10V, Capacitor_Tantalum_SMD:CP_EIA-7343-31_Kemet-D_Pad2.25x2.55mm_HandSolder, B.Cu at (106.8, 46.0)
- added D7: SS310, Diode_SMD:D_SMA, B.Cu at (46.2, 55.5)
- added L1: 68uH, Inductor_SMD:L_7.3x7.3_H3.5, B.Cu at (45.2, 63.7)
- added R1: 10K, Resistor_SMD:R_1206_3216Metric, B.Cu at (255.7, 66.2)
- added R7: 360R, Resistor_SMD:R_1206_3216Metric, B.Cu at (27.8, 59.5)
- added RV2: 10K, Potentiometer_THT:Potentiometer_Bourns_3296W_Vertical, B.Cu at (30.9, 76.8)
- added U11: KA78M05_TO252, Package_TO_SOT_SMD:TO-252-2, B.Cu at (114.8, 44.9)
- added U12: LM2596S-ADJ, Package_TO_SOT_SMD:TO-263-5_TabPin6, B.Cu at (35.5, 44.6)
- added U13: LD1117S33TR_SOT223, Package_TO_SOT_SMD:SOT-223-3_TabPin2, B.Cu at (114.0, 59.6)
- added U14: DW01A, Package_TO_SOT_SMD:SOT-23-6, B.Cu at (80.4, 50.0)
- C1, Q1, R5, R6, RV1, U1: moved to B.Cu
- C4: value C_Polarized_Small -> 10nF/50V; footprint Capacitor_SMD:CP_Elec_8x10 -> Capacitor_SMD:C_1206_3216Metric_Pad1.33x1.80mm_HandSolder; moved to B.Cu
- moved C1 205.1 mm to (260.2, 64.7), turned to 90 degrees
- moved Q1 203.8 mm to (225.8, 42.9), turned to 180 degrees
- moved RV1 163.9 mm to (182.5, 38.8)
- moved R6 162.1 mm to (230.2, 42.8)
- moved R5 156.7 mm to (234.5, 42.8)
- moved C4 113.1 mm to (129.2, 46.1), turned to 90 degrees
- moved U1 41.7 mm to (269.5, 87.0), turned to 90 degrees
- moved U2 38.3 mm to (182.8, 52.6), turned to 90 degrees
- moved C2 26.7 mm to (200.0, 52.9), turned to -90 degrees
- moved C3 19.4 mm to (195.0, 52.8), turned to -90 degrees
Connections:
- C4 pad 1: unconnected-(C4-Pad1) -> VCC-INT
- C4 pad 2: unconnected-(C4-Pad2) -> GND
Routing:
- net B: track 332.1 -> 0.00 mm, vias 5 -> 0
- net A: track 327.9 -> 0.00 mm, vias 5 -> 0
- net DP: track 324.2 -> 0.00 mm, vias 5 -> 0
- net F: track 316.8 -> 0.00 mm, vias 5 -> 0
- net G: track 312.1 -> 0.00 mm, vias 5 -> 0
- net F1: track 24.1 -> 0.00 mm, vias 1 -> 0
- net Net-(D1-K): track 19.8 -> 0.00 mm
- net Net-(D3-K): track 19.7 -> 0.00 mm
- net Net-(D2-K): track 19.7 -> 0.00 mm
- net E: track 16.2 -> 0.00 mm, vias 1 -> 0
- net D: track 15.0 -> 0.00 mm, vias 1 -> 0
- net C: track 14.3 -> 0.00 mm, vias 1 -> 0
- net M2: track 11.1 -> 0.00 mm
- net M1: track 11.1 -> 0.00 mm
- net H2: track 11.1 -> 0.00 mm
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- added copper zone on B.Cu, net GND
- added copper zone on F.Cu, net GND
Other:
- board size 270 x 120 mm -> 270 x 80 mm
- board text removed: "${REFERENCE}"

Commit message: Schematic updated
Parts:
- added BT1: Battery_Cell, Battery:BatteryHolder_ComfortableElectronic_CH273-2450_1x2450, B.Cu at (311.8, 170.9)
- added C16: 100nF/50V, Capacitor_SMD:C_1206_3216Metric_Pad1.33x1.80mm_HandSolder, B.Cu at (132.8, 99.9)
- added C17: 100nF/50V, Capacitor_SMD:C_1206_3216Metric_Pad1.33x1.80mm_HandSolder, B.Cu at (297.0, 147.3)
- added C18: 100nF/50V, Capacitor_SMD:C_1206_3216Metric_Pad1.33x1.80mm_HandSolder, B.Cu at (313.2, 180.6)
- added C19: 100nF/50V, Capacitor_SMD:C_1206_3216Metric_Pad1.33x1.80mm_HandSolder, F.Cu at (105.8, 184.0)
- added C20: 470uF/10V, Capacitor_Tantalum_SMD:CP_EIA-7343-31_Kemet-D_Pad2.25x2.55mm_HandSolder, F.Cu at (108.0, 172.8)
- added D8: LED_Dual_KAK, LED_THT:LED_D3.0mm-3, B.Cu at (120.8, 101.9)
- added DS1: WC1602A, Display:WC1602A, B.Cu at (159.6, 163.3)
- added J4: USB_B, Connector_USB:USB_B_Lumberg_2411_02_Horizontal, B.Cu at (329.6, 174.2)
- added Q2: FS8205A, Package_SO:TSSOP-8_3x3mm_P0.65mm, B.Cu at (130.6, 86.6)
- added R10: 100, Resistor_SMD:R_1206_3216Metric, B.Cu at (127.3, 92.4)
- added R11: 1K2, Resistor_SMD:R_0805_2012Metric_Pad1.20x1.40mm_HandSolder, B.Cu at (112.0, 88.4)
- added R12: 1K, Resistor_SMD:R_0805_2012Metric_Pad1.20x1.40mm_HandSolder, B.Cu at (125.0, 87.6)
- added R13: 4K7, Resistor_SMD:R_1206_3216Metric, B.Cu at (307.4, 143.3)
- added R14: 4K7, Resistor_SMD:R_1206_3216Metric, B.Cu at (307.4, 139.8)
- added R15: 470R, Resistor_SMD:R_1206_3216Metric, B.Cu at (287.2, 141.5)
- added R16: 10K, Resistor_SMD:R_1206_3216Metric, B.Cu at (82.6, 176.3)
- added R17: 10K, Resistor_SMD:R_1206_3216Metric, B.Cu at (82.5, 183.0)
- added R18: 10K, Resistor_SMD:R_1206_3216Metric, B.Cu at (82.5, 179.8)
- added R8: 1K, Resistor_SMD:R_0805_2012Metric_Pad1.20x1.40mm_HandSolder, B.Cu at (116.8, 95.1)
- added R9: 1K, Resistor_SMD:R_0805_2012Metric_Pad1.20x1.40mm_HandSolder, B.Cu at (120.3, 95.1)
- added RV3: 20K, Potentiometer_SMD:Potentiometer_Vishay_TS53YL_Vertical, B.Cu at (176.4, 167.8)
- added RV4: 20K, Potentiometer_SMD:Potentiometer_Vishay_TS53YL_Vertical, F.Cu at (107.3, 179.0)
- added SW1: RotaryEncoder-SW, Rotary_Encoder:RotaryEncoder_Bourns_Horizontal_PEC12R-2x17F-Sxxxx, B.Cu at (73.1, 181.8)
- added U15: DW01A, Package_TO_SOT_SMD:SOT-23-6, B.Cu at (126.9, 99.9)
- added U16: DS3231M, Package_SO:SOIC-16W_7.5x10.3mm_P1.27mm, B.Cu at (296.9, 138.5)
- added U17: MAX7219, Package_SO:SOIC-24W_7.5x15.4mm_P1.27mm, F.Cu at (96.4, 178.5)
- added U18: SA15-11SRWA, 7-segment-led:FYS-12011A, F.Cu at (101.8, 139.0)
- added U19: SA15-11SRWA, 7-segment-led:FYS-12011A, F.Cu at (131.8, 139.0)
- added U20: SA15-11SRWA, 7-segment-led:FYS-12011A, F.Cu at (161.9, 139.0)
- added U21: SA15-11SRWA, 7-segment-led:FYS-12011A, F.Cu at (192.1, 139.0)
- added U22: SA15-11SRWA, 7-segment-led:FYS-12011A, F.Cu at (222.2, 139.0)
- added U23: SA15-11SRWA, 7-segment-led:FYS-12011A, F.Cu at (252.2, 139.0)
- added U24: SA15-11SRWA, 7-segment-led:FYS-12011A, F.Cu at (282.4, 139.0)
- added U25: SA15-11SRWA, 7-segment-led:FYS-12011A, F.Cu at (312.4, 139.0)
- U14: value DW01A -> TP4056; footprint Package_TO_SOT_SMD:SOT-23-6 -> TP4056:TP4056-42-ESOP8_TPW
- moved U1 76.1 mm to (326.7, 137.1)
- moved C13 71.9 mm to (78.3, 97.1), turned to -90 degrees
- moved L1 71.9 mm to (105.5, 102.9), turned to 180 degrees
- moved U12 71.6 mm to (94.4, 85.5)
- moved C15 71.5 mm to (164.3, 101.1)
- moved C5 71.5 mm to (93.6, 106.9)
- moved C1 71.3 mm to (318.5, 105.8)
- moved C2 71.3 mm to (258.3, 94.0)
- moved C3 71.3 mm to (253.3, 93.9)
- moved D1 71.3 mm to (140.3, 86.1)
- moved D2 71.3 mm to (208.3, 85.7)
- moved D3 71.3 mm to (276.3, 85.7)
- moved D4 71.3 mm to (138.3, 107.7)
- moved D5 71.3 mm to (206.3, 107.1)
- moved D6 71.3 mm to (274.3, 107.1)
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Connections:
- C10 pad 1: VCC-INT -> +BATT
- C11 pad 1: VCC-INT -> +BATT
- C4 pad 1: VCC-INT -> +BATT
- C6 pad 1: VCC-INT -> +BATT
- U1 pad 15: unconnected-(U1-IO3-Pad15) -> D6
- U1 pad 16: unconnected-(U1-IO46-Pad16) -> ROT-CLK
- U1 pad 24: unconnected-(U1-IO47-Pad24) -> ROT-DT
- U1 pad 25: unconnected-(U1-IO48-Pad25) -> ROT-SW
- U1 pad 26: unconnected-(U1-IO45-Pad26) -> LOAD-SC
- U1 pad 38: unconnected-(U1-IO2-Pad38) -> D5
- U1 pad 39: unconnected-(U1-IO1-Pad39) -> D4
- U1 pad 4: unconnected-(U1-IO4-Pad4) -> D7
- U1 pad 5: unconnected-(U1-IO5-Pad5) -> CE
- U1 pad 6: unconnected-(U1-IO6-Pad6) -> RS
- U11 pad 1: VCC-INT -> +BATT
- U13 pad 3: VCC-INT -> +BATT
- U14 pad 1: unconnected-(U14-OD-Pad1) -> GND
- U14 pad 2: unconnected-(U14-CS-Pad2) -> Net-(U14-PROG)
- U14 pad 3: unconnected-(U14-OC-Pad3) -> GND
- U14 pad 4: unconnected-(U14-TD-Pad4) -> CHARGER
- U14 pad 5: unconnected-(U14-VCC-Pad5) -> +BATT
- U14 pad 6: unconnected-(U14-GND-Pad6) -> Net-(U14-*STDBY)
Routing:
- net +5V: track 0.00 -> 494.8 mm, vias 0 -> 6
- net +3.3V: track 0.00 -> 411.9 mm, vias 0 -> 4
- net SC-8: track 0.00 -> 296.6 mm
- net A: track 0.00 -> 293.0 mm, vias 0 -> 5
- net ROT-CLK: track 0.00 -> 292.9 mm
- net SC-C: track 0.00 -> 291.5 mm, vias 0 -> 1
- net SCK: track 0.00 -> 289.0 mm, vias 0 -> 3
- net MOSI: track 0.00 -> 284.1 mm, vias 0 -> 1
- net DP: track 0.00 -> 283.3 mm, vias 0 -> 2
- net SC-D: track 0.00 -> 282.4 mm, vias 0 -> 2
- net ROT-SW: track 0.00 -> 282.2 mm, vias 0 -> 1
- net F: track 0.00 -> 279.4 mm, vias 0 -> 1
- net SC-DP: track 0.00 -> 276.5 mm, vias 0 -> 1
- net SC-E: track 0.00 -> 275.4 mm, vias 0 -> 3
- net B: track 0.00 -> 271.7 mm, vias 0 -> 2
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Other:
- board size 270 x 80 mm -> 270 x 135.9 mm

Commit message: change page structure
Parts:
- removed U11: KA78M05_TO252, Package_TO_SOT_SMD:TO-252-2
- added D3: LED, LED_THT:LED_D10.0mm, F.Cu at (137.5, 68.0)
- added D6: LED, LED_THT:LED_D10.0mm, F.Cu at (273.7, 68.0)
- added J2: Serial, Connector_JST:JST_XH_B5B-XH-AM_1x05_P2.50mm_Vertical, F.Cu at (321.5, 178.0)
- added Q2: 2N2222, Package_TO_SOT_SMD:SOT-23, F.Cu at (265.1, 68.0)
- added R10: 100, Resistor_SMD:R_1206_3216Metric, B.Cu at (147.5, 68.0)
- added R12: 100, Resistor_SMD:R_1206_3216Metric, B.Cu at (283.5, 68.0)
- added R6: 100, Resistor_SMD:R_1206_3216Metric, F.Cu at (256.5, 68.0)
- added R8: 10K, Resistor_SMD:R_1206_3216Metric, F.Cu at (260.5, 68.0)
- C10, C4, C5: value 10nF/50V -> 100nF/50V
- C11: value 100uF/10V -> 220uF/10V
- C13: value 220uF/25V -> 100uF/10V
- C14: value 100nF/50V -> 10nF/50V
- C15, C9: value 220uF/10V -> 220uF/25V
- C6: value 100uF/10V -> 10nF/50V; footprint Capacitor_Tantalum_SMD:CP_EIA-7343-31_Kemet-D_Pad2.25x2.55mm_HandSolder -> Capacitor_SMD:C_1206_3216Metric_Pad1.33x1.80mm_HandSolder
- C7: value 220uF/25V -> 10nF/50V; footprint Capacitor_Tantalum_SMD:CP_EIA-7343-31_Kemet-D_Pad2.25x2.55mm_HandSolder -> Capacitor_SMD:C_1206_3216Metric_Pad1.33x1.80mm_HandSolder
- C8: value 100nF/50V -> 100uF/10V; footprint Capacitor_SMD:C_1206_3216Metric_Pad1.33x1.80mm_HandSolder -> Capacitor_Tantalum_SMD:CP_EIA-7343-31_Kemet-D_Pad2.25x2.55mm_HandSolder
- D7: value SS310 -> LED; footprint Diode_SMD:D_SMA -> LED_THT:LED_D3.0mm_FlatTop
- D8: value LED_Dual_KAK -> LED; footprint LED_THT:LED_D3.0mm-3 -> LED_THT:LED_D3.0mm_FlatTop
- Q2: value FS8205A -> 2N2222; footprint Package_SO:TSSOP-8_3x3mm_P0.65mm -> Package_TO_SOT_SMD:SOT-23
- R10: moved to F.Cu
- R11: value 1K2 -> 470R; footprint Resistor_SMD:R_0805_2012Metric_Pad1.20x1.40mm_HandSolder -> Resistor_SMD:R_1206_3216Metric
- R12: value 1K -> 100; footprint Resistor_SMD:R_0805_2012Metric_Pad1.20x1.40mm_HandSolder -> Resistor_SMD:R_1206_3216Metric
- R5: value 10K -> 100
- R7: value 360R -> 10K
- R8: value 1K -> 10K; footprint Resistor_SMD:R_0805_2012Metric_Pad1.20x1.40mm_HandSolder -> Resistor_SMD:R_1206_3216Metric
- R9: value 1K -> 470R; footprint Resistor_SMD:R_0805_2012Metric_Pad1.20x1.40mm_HandSolder -> Resistor_SMD:R_1206_3216Metric; moved to F.Cu
- RV2: value 10K -> 20K; footprint Potentiometer_THT:Potentiometer_Bourns_3296W_Vertical -> Potentiometer_SMD:Potentiometer_Vishay_TS53YL_Vertical
- U12: value LM2596S-ADJ -> KA78M05_TO252; footprint Package_TO_SOT_SMD:TO-263-5_TabPin6 -> Package_TO_SOT_SMD:TO-252-2
- U13: value LD1117S33TR_SOT223 -> LM2596S-ADJ; footprint Package_TO_SOT_SMD:SOT-223-3_TabPin2 -> Package_TO_SOT_SMD:TO-263-5_TabPin6
- U14: value TP4056 -> LD1117S33TR_SOT223; footprint TP4056:TP4056-42-ESOP8_TPW -> Package_TO_SOT_SMD:SOT-223-3_TabPin2
- moved R9 101.3 mm to (220.7, 108.5)
- moved R10 66.2 mm to (193.5, 92.4), turned to 0 degrees
- renumbered C17 to C4, C18 to C5, D4 to D2, D2 to D4, D3 to D7, D6 to D8, J4 to J1, R3 to R11, R4 to R13, R13 to R14, R14 to R15, R15 to R16, R16 to R2, R17 to R3, R18 to R4, R6 to R7, R2 to R9, RV3 to RV2, U6 to U10, U9 to U3, U10 to U4, U7 to U4, U8 to U5, U16 to U5, U4 to U6, U5 to U8
Connections:
- C10 pad 1: +BATT -> +5V
- C11 pad 1: +BATT -> +5V
- C12 pad 1: CHARGER -> +BATT
- C13 pad 1: CHARGER -> +BATT
- C14 pad 1: +3.3V -> CHARGER
- C15 pad 1: +3.3V -> CHARGER
- C16 pad 1: -BATT -> +3.3V
- C16 pad 2: Net-(U15-VCC) -> GND
- C4 pad 1: +BATT -> +3.3V
- C5 pad 1: +7-24V -> Net-(BT1-+)
- C8 pad 1: +5V -> +BATT
- C9 pad 1: +5V -> +7-24V
- D2 pad 1: Net-(D4-K) (its old number) -> Net-(D2-K)
- D4 pad 2: Net-(D2-A) -> Net-(D4-A)
- D5 pad 1: Net-(D4-K) (its old number) -> Net-(D2-K)
- D7 pad 1: Net-(D3-K) -> Net-(D7-K)
- D7 pad 2: Net-(D3-A) -> Net-(D7-A)
- D7 pad 2: GND -> Net-(D7-A)
- D8 pad 1: Net-(D4-K) (its old number) -> Net-(D2-K)
- D8 pad 2: Net-(D3-K) -> Net-(D7-K)
- D8 pad 1: Net-(D8-K1) -> Net-(D2-K)
- D8 pad 2: CHARGER -> Net-(D7-K)
- L1 pad 1: Net-(D7-K) -> Net-(D9-K)
- Q1 pad 3: Net-(D4-K) (its old number) -> Net-(D2-K)
- Q2 pad 1: unconnected-(Q2-Pad1)_1 -> Net-(Q2-B)
- Q2 pad 2: -BATT -> GND
- Q2 pad 3: -BATT -> Net-(D3-K)
- R10 pad 1: +BATT -> +5V
- R10 pad 2: Net-(U15-VCC) -> Net-(D3-A)
- R11 pad 2: Net-(D2-A) -> Net-(D4-A)
- R11 pad 1: Net-(U14-PROG) -> +5V
- R11 pad 2: GND -> Net-(D4-A)
- R12 pad 1: Net-(U15-CS) -> +5V
- R12 pad 2: GND -> Net-(D6-A)
- R13 pad 2: Net-(D3-A) -> Net-(D7-A)
- R7 pad 1: Net-(U12-FB) -> Net-(Q1-B)
- R8 pad 1: Net-(D8-K2) -> Net-(Q2-B)
- R8 pad 2: Net-(U14-*CHRG) -> GND
- R9 pad 1: Net-(D8-K1) -> +5V
- R9 pad 2: Net-(U14-*STDBY) -> Net-(D1-A)
- RV2 pad 1: Net-(U12-FB) -> +5V
- RV2 pad 2: Net-(U12-FB) -> +5V
- RV2 pad 3: CHARGER -> Net-(DS1-VO)
- U1 pad 18: unconnected-(U1-IO10-Pad18) -> SW1
- U1 pad 22: unconnected-(U1-IO14-Pad22) -> SW2
- U1 pad 36: unconnected-(U1-RXD0-Pad36) -> RX0
- U1 pad 37: unconnected-(U1-TXD0-Pad37) -> TX0
- U1 pad 7: unconnected-(U1-IO7-Pad7) -> CLAP-LED
- U1 pad 8: unconnected-(U1-IO15-Pad8) -> SW3
- U1 pad 9: unconnected-(U1-IO16-Pad9) -> SW4
- U12 pad 1: +7-24V -> +BATT
- U12 pad 2: Net-(D7-K) -> GND
- U12 pad 3: GND -> +5V
- U13 pad 1: GND -> +7-24V
- U13 pad 2: +3.3V -> Net-(D9-K)
- U13 pad 3: +BATT -> GND
- U14 pad 2: Net-(U14-PROG) -> +3.3V
- U14 pad 3: GND -> +BATT
- U19 pad 1: SC-2 -> SC-5
- U19 pad 5: SC-2 -> SC-5
- U20 pad 1: SC-3 -> SC-2
- U20 pad 5: SC-3 -> SC-2
- U21 pad 1: SC-4 -> SC-6
- U21 pad 5: SC-4 -> SC-6
- U22 pad 1: SC-5 -> SC-3
- U22 pad 5: SC-5 -> SC-3
- U23 pad 1: SC-6 -> SC-7
- U23 pad 5: SC-6 -> SC-7
- U24 pad 1: SC-7 -> SC-4
- U24 pad 5: SC-7 -> SC-4
Routing:
- net +5V: track 494.8 -> 0.00 mm, vias 6 -> 0
- net +3.3V: track 411.9 -> 0.00 mm, vias 4 -> 0
- net SC-8: track 296.6 -> 0.00 mm
- net A: track 293.0 -> 0.00 mm, vias 5 -> 0
- net ROT-CLK: track 292.9 -> 0.00 mm
- net SC-C: track 291.5 -> 0.00 mm, vias 1 -> 0
- net SCK: track 289.0 -> 0.00 mm, vias 3 -> 0
- net MOSI: track 284.1 -> 0.00 mm, vias 1 -> 0
- net DP: track 283.3 -> 0.00 mm, vias 2 -> 0
- net SC-D: track 282.4 -> 0.00 mm, vias 2 -> 0
- net ROT-SW: track 282.2 -> 0.00 mm, vias 1 -> 0
- net F: track 279.4 -> 0.00 mm, vias 1 -> 0
- net SC-DP: track 276.5 -> 0.00 mm, vias 1 -> 0
- net SC-E: track 275.4 -> 0.00 mm, vias 3 -> 0
- net B: track 271.7 -> 0.00 mm, vias 2 -> 0
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
Commit message: schematic and board layout finished
Parts:
- removed the C4 at (187.5, 86.8)
- removed the C5 at (93.6, 106.9)
- removed the C6 at (181.5, 86.7)
- removed the C7 at (93.5, 100.4)
- removed the D3 at (137.5, 68.0)
- removed the D6 at (273.7, 68.0)
- removed the Q2 at (130.6, 86.6)
- removed the R10 at (193.5, 92.4)
- removed the R11 at (112.0, 88.4)
- removed the R12 at (125.0, 87.6)
- removed the R7 at (85.3, 100.6)
- removed the R8 at (116.8, 95.1)
- removed the R9 at (220.7, 108.5)
- removed the RV2 at (84.3, 107.4)
- removed the U12 at (94.4, 85.5)
- removed the U13 at (172.0, 101.0)
- removed the U14 at (118.5, 88.9)
- removed the U15 at (126.9, 99.9)
- added C17: 10nF/50V, Capacitor_SMD:C_1206_3216Metric_Pad1.33x1.80mm_HandSolder, B.Cu at (201.5, 182.6)
- added C18: 100uF/10V, Capacitor_Tantalum_SMD:CP_EIA-7343-31_Kemet-D_Pad2.25x2.55mm_HandSolder, B.Cu at (207.8, 184.6)
- added C19: 100nF/50V, Capacitor_SMD:C_1206_3216Metric_Pad1.33x1.80mm_HandSolder, B.Cu at (224.9, 192.2)
- added C20: 220uF/10V, Capacitor_Tantalum_SMD:CP_EIA-7343-31_Kemet-D_Pad2.25x2.55mm_HandSolder, B.Cu at (226.8, 186.0)
- added C21: 100nF/50V, Capacitor_SMD:C_1206_3216Metric_Pad1.33x1.80mm_HandSolder, F.Cu at (182.8, 177.9)
- added D10: SS310, Diode_SMD:D_SMA, B.Cu at (260.5, 172.5)
- added D11: EXT, LED_SMD:LED_0201_0603Metric_Pad0.64x0.40mm_HandSolder, B.Cu at (245.5, 181.9)
- added D12: 5V, LED_SMD:LED_0201_0603Metric_Pad0.64x0.40mm_HandSolder, B.Cu at (197.8, 174.9)
- added D13: 3V3, LED_SMD:LED_0201_0603Metric_Pad0.64x0.40mm_HandSolder, B.Cu at (197.8, 180.9)
- added D14: 1N4148, Diode_SMD:D_PowerDI-123, F.Cu at (191.5, 178.0)
- added D9: LED_Dual_KAK, LED_THT:LED_D3.0mm-3, B.Cu at (324.5, 188.2)
- added J3: +8-24 Volt, Connector_BarrelJack:BarrelJack_GCT_DCJ200-10-A_Horizontal, F.Cu at (331.6, 190.8)
- added J4: Battery, Connector_JST:JST_XH_B2B-XH-AM_1x02_P2.50mm_Vertical, B.Cu at (237.2, 176.5)
- added J5: Mains, Connector_JST:JST_XH_B2B-XH-AM_1x02_P2.50mm_Vertical, B.Cu at (238.2, 190.2)
- added J6: Mains, Connector_JST:JST_XH_B2B-XH-AM_1x02_P2.50mm_Vertical, B.Cu at (327.1, 67.0)
- added J7: Timecode IN, Connector_Audio:Jack_3.5mm_CUI_SJ1-3525N_Horizontal, B.Cu at (187.2, 192.5)
- added J8: Timecode OUT, Connector_Audio:Jack_3.5mm_CUI_SJ1-3525N_Horizontal, B.Cu at (173.2, 192.5)
- added Q3: FS8205A, Package_SO:TSSOP-8_3x3mm_P0.65mm, F.Cu at (224.1, 177.8)
- added Q4: 2N2222, Package_TO_SOT_SMD:SOT-23, F.Cu at (189.2, 171.9)
- added R17: 100, Resistor_SMD:R_1206_3216Metric, F.Cu at (237.1, 168.5)
- added R18: 1K, Resistor_SMD:R_0805_2012Metric_Pad1.20x1.40mm_HandSolder, F.Cu at (317.2, 193.0)
- added R19: 1K, Resistor_SMD:R_0805_2012Metric_Pad1.20x1.40mm_HandSolder, F.Cu at (317.2, 189.0)
- added R20: 360R, Resistor_SMD:R_1206_3216Metric, B.Cu at (271.2, 178.1)
- added R21: 1K, Resistor_SMD:R_0805_2012Metric_Pad1.20x1.40mm_HandSolder, F.Cu at (218.2, 173.5)
- added R22: 1K2, Resistor_SMD:R_0805_2012Metric_Pad1.20x1.40mm_HandSolder, F.Cu at (243.1, 176.5)
- added R23: 180, Resistor_SMD:R_0805_2012Metric_Pad1.20x1.40mm_HandSolder, B.Cu at (245.0, 174.9)
- added R24: 180, Resistor_SMD:R_0805_2012Metric_Pad1.20x1.40mm_HandSolder, B.Cu at (201.5, 175.0)
- added R25: 180, Resistor_SMD:R_0805_2012Metric_Pad1.20x1.40mm_HandSolder, B.Cu at (201.0, 188.2)
- added R26: 10K, Resistor_SMD:R_1206_3216Metric, B.Cu at (90.8, 182.4)
- added R27: 10K, Resistor_SMD:R_1206_3216Metric, B.Cu at (90.8, 185.7)
- added R28: 10K, Resistor_SMD:R_1206_3216Metric, B.Cu at (90.8, 189.0)
- added R29: 10K, Resistor_SMD:R_1206_3216Metric, B.Cu at (90.8, 192.3)
- added R30: 10K, Resistor_SMD:R_1206_3216Metric, B.Cu at (332.9, 67.5)
- added R31: 100, Resistor_SMD:R_1206_3216Metric, F.Cu at (194.2, 172.0)
- added R32: 10K, Resistor_SMD:R_1206_3216Metric, F.Cu at (187.0, 178.0)
- added R33: 1K8, Resistor_SMD:R_1206_3216Metric, F.Cu at (172.2, 177.7)
- added R34: 5K6, Resistor_SMD:R_1206_3216Metric, F.Cu at (176.5, 177.7)
- added RV4: 10K, Potentiometer_THT:Potentiometer_Bourns_3296W_Vertical, B.Cu at (270.1, 171.0)
- added SW2: 1, Button_Switch_THT:SW_PUSH-12mm, B.Cu at (153.0, 193.8)
- added SW3: 1, Button_Switch_THT:SW_PUSH-12mm, B.Cu at (137.5, 193.8)
- added SW4: 1, Button_Switch_THT:SW_PUSH-12mm, B.Cu at (121.9, 193.8)
- added SW5: 1, Button_Switch_THT:SW_PUSH-12mm, B.Cu at (106.4, 193.8)
- added U21: LM2596S-ADJ, Package_TO_SOT_SMD:TO-263-5_TabPin6, B.Cu at (262.7, 186.7)
- added U22: DW01A, Package_TO_SOT_SMD:SOT-23-6, F.Cu at (223.8, 170.7)
- added U23: TP4056, TP4056:TP4056-42-ESOP8_TPW, F.Cu at (243.1, 169.5)
- added U24: KA78M05_TO252, Package_TO_SOT_SMD:TO-252-2, B.Cu at (216.5, 170.2)
- added U25: LD1117S33TR_SOT223, Package_TO_SOT_SMD:SOT-223-3_TabPin2, B.Cu at (216.4, 184.7)
- C10: value 100nF/50V -> 10nF/50V
- C11: value 220uF/10V -> 220uF/25V
- C12: value 10nF/50V -> 100nF/50V; moved to F.Cu
- C13, C8: value 100uF/10V -> 10nF/50V; footprint Capacitor_Tantalum_SMD:CP_EIA-7343-31_Kemet-D_Pad2.25x2.55mm_HandSolder -> Capacitor_SMD:C_1206_3216Metric_Pad1.33x1.80mm_HandSolder
- C14: value 10nF/50V -> 100uF/10V; footprint Capacitor_SMD:C_1206_3216Metric_Pad1.33x1.80mm_HandSolder -> Capacitor_Tantalum_SMD:CP_EIA-7343-31_Kemet-D_Pad2.25x2.55mm_HandSolder
- C15: value 220uF/25V -> 100nF/50V; footprint Capacitor_Tantalum_SMD:CP_EIA-7343-31_Kemet-D_Pad2.25x2.55mm_HandSolder -> Capacitor_SMD:C_1206_3216Metric_Pad1.33x1.80mm_HandSolder
- C16: value 100nF/50V -> 220uF/10V; footprint Capacitor_SMD:C_1206_3216Metric_Pad1.33x1.80mm_HandSolder -> Capacitor_Tantalum_SMD:CP_EIA-7343-31_Kemet-D_Pad2.25x2.55mm_HandSolder
- C3: renamed from C5; moved to F.Cu
- C4: renamed from C19; moved to B.Cu
- C5: renamed from C20; moved to B.Cu
- D7, D8: footprint LED_THT:LED_D3.0mm_FlatTop -> LED_THT:LED_D10.0mm; moved to F.Cu
- J1: renamed from J2; moved to B.Cu
- RV2: renamed from RV4; moved to B.Cu
- U7: renamed from U17; moved to B.Cu
- moved C13 169.5 mm to (231.8, 168.9), turned to 90 degrees
- moved L1 167.0 mm to (260.6, 164.9), turned to 0 degrees
- moved C12 164.9 mm to (231.8, 168.3), turned to -90 degrees
- moved D8 156.3 mm to (273.5, 68.5), turned to 0 degrees
- moved C4 142.8 mm to (240.5, 136.4), turned to -90 degrees
- moved U7 132.9 mm to (222.7, 137.1), turned to 180 degrees
- moved C8 132.7 mm to (251.4, 182.0), turned to 0 degrees
- moved C9 132.2 mm to (249.4, 188.7), turned to 0 degrees
- moved C5 131.6 mm to (234.5, 136.8), turned to -90 degrees
- moved RV2 111.1 mm to (210.2, 137.2)
- moved C16 103.5 mm to (207.8, 171.2)
- moved C11 98.4 mm to (251.0, 169.0)
- moved C14 97.0 mm to (225.2, 171.2)
- moved C10 89.0 mm to (245.0, 166.8)
- moved C15 77.7 mm to (201.8, 169.2)
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- renumbered C4 to C2, C2 to C6, C3 to C7, D4 to D2, D7 to D3, D2 to D4, D8 to D6, J1 to J2, R13 to R10, R5 to R11, R7 to R12, R10 to R13, R12 to R14, R6 to R15, R8 to R16, R14 to R5, R15 to R6, R16 to R7, R9 to R8, R11 to R9, RV2 to RV1, RV1 to RV3, U24 to U10, U25 to U11, U3 to U12, U4 to U13, U5 to U14, U4 to U15, U2 to U16, U10 to U17, U8 to U18, U6 to U19, U5 to U2, U3 to U20, U18 to U3, U19 to U4, U20 to U5, U21 to U6, U22 to U8, U23 to U9
Connections:
- C10 pad 1: +5V -> CHARGER
- C11 pad 1: +5V -> CHARGER
- C12 pad 1: +BATT -> -BATT
- C12 pad 2: GND -> Net-(U22-VCC)
- C13 pad 1: +BATT -> VCC-INT
- C14 pad 1: CHARGER -> VCC-INT
- C15 pad 1: CHARGER -> +5V
- C16 pad 1: +3.3V -> +5V
- C8 pad 1: +BATT -> Net-(U21-VIN)
- C9 pad 1: +7-24V -> Net-(U21-VIN)
- D3 pad 1: Net-(D7-K) -> Net-(D3-K)
- D3 pad 2: Net-(D7-A) -> Net-(D3-A)
- D4 pad 1: Net-(D2-K) (its old number) -> Net-(D4-K)
- D5 pad 1: Net-(D2-K) (its old number) -> Net-(D4-K)
- D6 pad 1: Net-(D2-K) (its old number) -> Net-(D4-K)
- D6 pad 2: Net-(D7-K) -> Net-(D3-K)
- D8 pad 1: Net-(D2-K) (its old number) -> Net-(D7-K)
- D8 pad 2: Net-(D7-K) -> Net-(D8-A)
- Q1 pad 3: Net-(D2-K) (its old number) -> Net-(D4-K)
- Q2 pad 3: Net-(D3-K) -> Net-(D7-K)
- R10 pad 2: Net-(D7-A) -> Net-(D3-A)
- R13 pad 2: Net-(D3-A) -> Net-(D7-A)
- R14 pad 2: Net-(D6-A) -> Net-(D8-A)
- U10 pad 1: SC-4 -> SC-7
- U10 pad 5: SC-4 -> SC-7
- U12 pad 1: F1 -> H1
- U12 pad 5: F1 -> H1
- U13 pad 1: F2 -> H2
- U13 pad 5: F2 -> H2
- U14 pad 1: S2 -> M1
- U14 pad 5: S2 -> M1
- U15 pad 1: S1 -> M2
- U15 pad 5: S1 -> M2
- U17 pad 1: M2 -> S1
- U17 pad 5: M2 -> S1
- U18 pad 1: M1 -> S2
- U18 pad 5: M1 -> S2
- U19 pad 1: H2 -> F1
- U19 pad 5: H2 -> F1
- U20 pad 1: H1 -> F2
- U20 pad 5: H1 -> F2
- U4 pad 1: SC-5 -> SC-2
- U4 pad 5: SC-5 -> SC-2
- U5 pad 1: SC-2 -> SC-3
- U5 pad 5: SC-2 -> SC-3
- U6 pad 1: SC-6 -> SC-4
- U6 pad 5: SC-6 -> SC-4
- U8 pad 1: SC-3 -> SC-5
- U8 pad 5: SC-3 -> SC-5
- U9 pad 1: SC-7 -> SC-6
- U9 pad 5: SC-7 -> SC-6
