File: hardware/PCB/DigiSlatePlus.kicad_pcb (KiCad board)
At the start: 2 copper layers, 270 x 135.9 mm, 118 parts, among them J1 Serial, J2 USB_B, J3 +8-24 Volt, J4 Battery, J5 Mains, J6 Mains, J7 Timecode IN, J8 Timecode OUT, Q1 2N2222, Q2 2N2222, Q3 FS8205A, Q4 2N2222, SW1 RotaryEncoder-SW, SW2 1, SW3 1, SW4 1, SW5 1, U1 ESP32-S3-WROOM-1, U10 SA15-11SRWA, U11 SA15-11SRWA, U12 SA15-11SRWA, U13 SA15-11SRWA, U14 SA15-11SRWA, U15 SA15-11SRWA, U16 MAX7219, U17 SA15-11SRWA, U18 SA15-11SRWA, U19 SA15-11SRWA, U2 DS3231M, U20 SA15-11SRWA, U21 LM2596S-ADJ, U22 DW01A, U23 TP4056, U24 KA78M05_TO252, U25 LD1117S33TR_SOT223, U3 SA15-11SRWA, U4 SA15-11SRWA, U5 SA15-11SRWA, U6 SA15-11SRWA, U7 MAX7219, U8 SA15-11SRWA, U9 SA15-11SRWA

Commit message: first finished schematic version
Parts:
- added J10: IO7, Connector_PinHeader_1.00mm:PinHeader_1x01_P1.00mm_Vertical, B.Cu at (330.2, 158.5)
- added J9: MISO, Connector_PinHeader_1.00mm:PinHeader_1x01_P1.00mm_Vertical, B.Cu at (302.0, 116.5)
- added SW6: BOOT, Button_Switch_SMD:SW_Push_SPST_NO_Alps_SKRK, B.Cu at (325.1, 120.5)
- D11: footprint LED_SMD:LED_0201_0603Metric_Pad0.64x0.40mm_HandSolder -> LED_THT:LED_D3.0mm
- D12, D13: footprint LED_SMD:LED_0201_0603Metric_Pad0.64x0.40mm_HandSolder -> LED_SMD:LED_0603_1608Metric
- R18, R19: moved to B.Cu
- moved D11 80.0 mm to (325.0, 190.8), turned to 180 degrees
- moved R23 74.7 mm to (318.0, 190.8), turned to -90 degrees
- moved D9 13.3 mm to (311.2, 188.4)
- moved R18 13.3 mm to (304.0, 193.2), turned to 0 degrees
- moved R19 13.3 mm to (304.0, 189.2), turned to 0 degrees
- turned C8 to 180 degrees
Connections:
- R15 pad 1: CLAP-LED -> FLASH-LED
- U1 pad 27: BOOT -> Net-(U1-IO0)
- U1 pad 7: CLAP-LED -> IO7
Routing:
- net +5V: track 0.00 -> 550.7 mm, vias 0 -> 4
- net +3.3V: track 0.00 -> 487.1 mm, vias 0 -> 2
- net DP: track 0.00 -> 298.5 mm
- net SW2: track 0.00 -> 296.8 mm, vias 0 -> 2
- net SW3: track 0.00 -> 278.9 mm, vias 0 -> 1
- net F: track 0.00 -> 278.4 mm, vias 0 -> 1
- net A: track 0.00 -> 274.4 mm, vias 0 -> 3
- net B: track 0.00 -> 274.3 mm, vias 0 -> 2
- net E: track 0.00 -> 273.8 mm
- net G: track 0.00 -> 272.3 mm, vias 0 -> 2
- net ROT-CLK: track 0.00 -> 271.9 mm, vias 0 -> 1
- net C: track 0.00 -> 269.5 mm, vias 0 -> 1
- net SW4: track 0.00 -> 268.0 mm, vias 0 -> 1
- net D: track 0.00 -> 267.7 mm, vias 0 -> 2
- net ROT-SW: track 0.00 -> 265.8 mm, vias 0 -> 2
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
Commit message: final 1.0 board version
Parts:
- removed D8: LED, LED_THT:LED_D10.0mm
- removed J5: Mains, Connector_JST:JST_XH_B2B-XH-AM_1x02_P2.50mm_Vertical
- removed R14: 100, Resistor_SMD:R_1206_3216Metric
- added Hole1: MountingHole_3.2mm_M3_Pad, MountingHole:MountingHole_3.2mm_M3_Pad, F.Cu at (77.0, 71.0)
- added Hole2: MountingHole_3.2mm_M3_Pad, MountingHole:MountingHole_3.2mm_M3_Pad, F.Cu at (207.0, 71.0)
- added Hole3: MountingHole_3.2mm_M3_Pad, MountingHole:MountingHole_3.2mm_M3_Pad, F.Cu at (337.0, 71.0)
- added Hole4: MountingHole_3.2mm_M3_Pad, MountingHole:MountingHole_3.2mm_M3_Pad, F.Cu at (337.0, 201.0)
- added Hole5: MountingHole_3.2mm_M3_Pad, MountingHole:MountingHole_3.2mm_M3_Pad, F.Cu at (207.0, 201.0)
- added Hole6: MountingHole_3.2mm_M3_Pad, MountingHole:MountingHole_3.2mm_M3_Pad, F.Cu at (77.0, 201.0)
- added REF**: KiCad-Logo2_6mm_SilkScreen, Symbol:KiCad-Logo2_6mm_SilkScreen, F.Cu at (286.0, 196.0)
- added SW7: SW_DPDT_x2, Button_Switch_THT:SW_Slide_SPDT_Angled_CK_OS102011MA1Q, B.Cu at (242.4, 203.7)
- Q2, R10, R15, R16, R8, R9: moved to B.Cu
- SW2, SW3, SW4, SW5: footprint Button_Switch_THT:SW_PUSH-12mm -> Button_Switch_THT:SW_Tactile_Straight_KSA0Axx1LFTR
- U21: footprint Package_TO_SOT_SMD:TO-263-5_TabPin6 -> Package_TO_SOT_SMD:TO-263-5_TabPin3
- moved Q2 200.4 mm to (81.8, 149.0), turned to 90 degrees
- moved R16 198.5 mm to (81.7, 154.4), turned to 180 degrees
- moved R15 197.2 mm to (76.2, 147.8), turned to -90 degrees
- moved R13 112.0 mm to (76.2, 154.5), turned to 90 degrees
- moved D7 87.6 mm to (80.8, 135.3), turned to -90 degrees
- moved R30 66.1 mm to (275.1, 99.7), turned to 180 degrees
- moved J6 58.2 mm to (275.6, 93.9), turned to 90 degrees
- moved R26 53.9 mm to (141.8, 199.8), turned to 90 degrees
- moved R27 38.0 mm to (126.0, 199.8), turned to 90 degrees
- moved R28 22.5 mm to (110.5, 199.8), turned to 90 degrees
- moved DS1 16.3 mm to (158.5, 161.5)
- moved SW4 11.2 mm to (114.4, 202.1), turned to 0 degrees
- moved SW5 11.2 mm to (98.8, 202.0), turned to 0 degrees
- moved D14 11.0 mm to (182.2, 183.9)
- moved SW3 10.9 mm to (130.4, 202.0), turned to 0 degrees
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Routing:
- net GND: track 0.00 -> 941.0 mm, vias 0 -> 5
- net FLASH-LED: track 106.3 -> 257.0 mm, vias 1 -> 2
- net Net-(D7-K): track 137.2 -> 13.5 mm
- net SCK: track 265.0 -> 166.2 mm, vias 3 -> 2
- net SW2: track 296.8 -> 233.2 mm
- net SC-D: track 231.9 -> 293.8 mm, vias 2 -> 0
- net SW1: track 259.8 -> 203.4 mm
- net DP: track 298.5 -> 259.1 mm, vias 0 -> 1
- net SW3: track 278.9 -> 244.7 mm
- net SC-2: track 139.0 -> 107.3 mm
- net SC-DP: track 261.7 -> 231.5 mm, vias 2 -> 0
- net SC-E: track 235.9 -> 265.1 mm, vias 3 -> 1
- net SC-C: track 235.1 -> 260.7 mm, vias 1 -> 3
- net Net-(D10-K): track 43.7 -> 24.3 mm
- net Net-(U21-VIN): track 106.6 -> 87.7 mm, vias 0 -> 1
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Other:
- board size 270 x 135.9 mm -> 270 x 140 mm
- board text added: "DigiSlate+"
- board text added: "V1.0"
- board text added: "https://digislateplus.github.io"
