File: hardware/PCB/tc_display.kicad_sch (KiCad schematic)
At the start: 43 parts, among them Q1 2N2222, Q2 2N2222, U10 SA15-11SRWA, U11 SA15-11SRWA, U12 SA15-11SRWA, U13 SA15-11SRWA, U14 SA15-11SRWA, U15 SA15-11SRWA, U16 MAX7219, U17 SA15-11SRWA, U18 SA15-11SRWA, U19 SA15-11SRWA, U20 SA15-11SRWA, U3 SA15-11SRWA, U4 SA15-11SRWA, U5 SA15-11SRWA, U6 SA15-11SRWA, U7 MAX7219, U8 SA15-11SRWA, U9 SA15-11SRWA

Commit message: first finished schematic version
Connections:
- net CLAP-LED renamed FLASH-LED
Changed lines of the file:
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@@
 		)
 	)
-	(global_label "CLAP-LED"
+	(global_label "FLASH-LED"
 		(shape input)
 		(at 220.98 104.14 90)
@@
 		)
 		(property "Intersheetrefs" "${INTERSHEET_REFS}"
-			(at 220.98 91.4786 90)
+			(at 220.98 90.39 90)
 			(effects
 				(font

Commit message: final 1.0 board version
Parts:
- removed D8: LED, LED_THT:LED_D10.0mm, symbol Device:LED
- removed R14: 100, Resistor_SMD:R_1206_3216Metric, symbol Device:R
Other:
- title: (none) -> DigiSlate+
- moved on the sheet: D7, R13
